File: sync.kicad_sch (KiCad schematic)
At the start: 5 parts, among them J1 Conn_01x04_Male, J2 Conn_01x04_Male, U1 LTC1485

Commit message: update
Parts:
- U1: footprint Package_DIP:DIP-8_W7.62mm -> Package_SO:SO-8_3.9x4.9mm_P1.27mm
Connections:
- net GND1: now also J1.4 (Pin_4); no longer J1.2 (Pin_2)
- net VCC: now also J1.3 (Pin_3); no longer J1.1 (Pin_1)
- net SIGNAL: now reaches U1.4 (DI)
- net SIGNAL: now also J1.2 (Pin_2); no longer J1.3 (Pin_3)
- net at R1.2, U1.6 (A): now also J2.1 (Pin_1), J2.3 (Pin_3); no longer J2.2 (Pin_2)
- net at R1.1, U1.7 (B): now also J2.2 (Pin_2), J2.4 (Pin_4); no longer J2.3 (Pin_3)
Other:
- moved on the sheet: J1, J2

Commit message: place route
Connections:
- net D+: now reaches R1.2, U1.6 (A)
- net D+: now also J2.2 (Pin_2), J2.4 (Pin_4); no longer J2.1 (Pin_1), J2.3 (Pin_3)
- net D-: now reaches R1.1, U1.7 (B)
- net D-: now also J2.1 (Pin_1), J2.3 (Pin_3); no longer J2.2 (Pin_2), J2.4 (Pin_4)

Commit message: add lidar-if
Parts:
- J2: footprint Connector_JST:JST_XA_S04B-XASK-1_1x04_P2.50mm_Horizontal -> Connector_JST:JST_XA_S04B-XASK-1N-BN_1x04_P2.50mm_Horizontal
Other:
- moved on the sheet: C1
Changed lines of the file:
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@@
     )
   )
-  (symbol (lib_id "power:GND1") (at 76.2 80.01 0) (unit 1)
-    (in_bom yes) (on_board yes) (dnp no) (fields_autoplaced)
-    (property "Reference" "#PWR04" (at 76.2 86.36 0)
-      (effects (font (size 1.27 1.27)) hide)
-    )
-    (property "Value" "GND1" (at 76.2 85.09 0)
-      (effects (font (size 1.27 1.27)))
-    )
-    (property "Footprint" "" (at 76.2 80.01 0)
-      (effects (font (size 1.27 1.27)) hide)
-    )
-    (property "Datasheet" "" (at 76.2 80.01 0)
+  (symbol (lib_id "power:GND1") (at 53.34 88.9 0) (unit 1)
+    (in_bom yes) (on_board yes) (dnp no) (fields_autoplaced)
+    (property "Reference" "#PWR04" (at 53.34 95.25 0)
+      (effects (font (size 1.27 1.27)) hide)
+    )
+    (property "Value" "GND1" (at 53.34 93.98 0)
+      (effects (font (size 1.27 1.27)))
+    )
+    (property "Footprint" "" (at 53.34 88.9 0)
+      (effects (font (size 1.27 1.27)) hide)
+    )
+    (property "Datasheet" "" (at 53.34 88.9 0)
       (effects (font (size 1.27 1.27)) hide)
     )
@@
     )
   )
-  (symbol (lib_id "pspice:CAP") (at 76.2 73.66 0) (unit 1)
-    (in_bom yes) (on_board yes) (dnp no) (fields_autoplaced)
-    (property "Reference" "C1" (at 81.28 72.3899 0)
-      (effects (font (size 1.27 1.27)) (justify left))
-    )
-    (property "Value" "0.1u" (at 81.28 74.9299 0)
-      (effects (font (size 1.27 1.27)) (justify left))
-    )
-    (property "Footprint" "Capacitor_SMD:C_0603_1608Metric" (at 76.2 73.66 0)
-      (effects (font (size 1.27 1.27)) hide)
-    )
-    (property "Datasheet" "~" (at 76.2 73.66 0)
+  (symbol (lib_id "pspice:CAP") (at 53.34 82.55 0) (unit 1)
+    (in_bom yes) (on_board yes) (dnp no) (fields_autoplaced)
+    (property "Reference" "C1" (at 58.42 81.2799 0)
+      (effects (font (size 1.27 1.27)) (justify left))
+    )
+    (property "Value" "0.1u" (at 58.42 83.8199 0)
+      (effects (font (size 1.27 1.27)) (justify left))
+    )
+    (property "Footprint" "Capacitor_SMD:C_0603_1608Metric" (at 53.34 82.55 0)
+      (effects (font (size 1.27 1.27)) hide)
+    )
+    (property "Datasheet" "~" (at 53.34 82.55 0)
       (effects (font (size 1.27 1.27)) hide)
     )
@@
     )
   )
-  (symbol (lib_id "power:VCC") (at 76.2 67.31 0) (unit 1)
-    (in_bom yes) (on_board yes) (dnp no) (fields_autoplaced)
-    (property "Reference" "#PWR03" (at 76.2 71.12 0)
-      (effects (font (size 1.27 1.27)) hide)
-    )
-    (property "Value" "VCC" (at 76.2 62.23 0)
-      (effects (font (size 1.27 1.27)))
-    )
-    (property "Footprint" "" (at 76.2 67.31 0)
-      (effects (font (size 1.27 1.27)) hide)
-    )
-    (property "Datasheet" "" (at 76.2 67.31 0)
+  (symbol (lib_id "power:VCC") (at 53.34 76.2 0) (unit 1)
+    (in_bom yes) (on_board yes) (dnp no) (fields_autoplaced)
+    (property "Reference" "#PWR03" (at 53.34 80.01 0)
+      (effects (font (size 1.27 1.27)) hide)
+    )
+    (property "Value" "VCC" (at 53.34 71.12 0)
+      (effects (font (size 1.27 1.27)))
+    )
+    (property "Footprint" "" (at 53.34 76.2 0)
+      (effects (font (size 1.27 1.27)) hide)
+    )
+    (property "Datasheet" "" (at 53.34 76.2 0)
       (effects (font (size 1.27 1.27)) hide)
     )
@@
       (effects (font (size 1.27 1.27)) (justify right) hide)
     )
-    (property "Footprint" "Connector_JST:JST_XA_S04B-XASK-1_1x04_P2.50mm_Horizontal" (at 135.89 58.42 0)
-      (effects (font (size 1.27 1.27)) hide)
-    )
+    (property "Footprint" "Connector_JST:JST_XA_S04B-XASK-1N-BN_1x04_P2.50mm_Horizontal" (at 135.89 58.42 0)
+      (effects (font (size 1.27 1.27)) hide)
+    )

Commit message: backup
Parts:
- added D1, D2: 12V, sync:SMA (DO-214AC), symbol sync:SMAJ12A-E3/61
- added JP1: SolderJumper_3_Open, Jumper:SolderJumper-3_P1.3mm_Open_Pad1.0x1.5mm, symbol Jumper:SolderJumper_3_Open
- added R2: 1K, Resistor_SMD:R_0603_1608Metric, symbol Device:R_US
- C1: footprint Capacitor_SMD:C_0603_1608Metric -> Jumper:SolderJumper-3_P1.3mm_Open_RoundedPad1.0x1.5mm
Connections:
- net D+: now also J2.1 (Pin_1), J2.3 (Pin_3), D2.1, JP1.2 (C); no longer J2.2 (Pin_2), J2.4 (Pin_4), R1.2
- net D-: now also J2.2 (Pin_2), J2.4 (Pin_4), D1.1, R2.1; no longer J2.1 (Pin_1), J2.3 (Pin_3)
- net GND1: now also D1.2, D2.2
- new net: JP1.1 (A), R2.2
- new net: JP1.3 (B), R1.2
Other:
- moved on the sheet: J2, R1

Commit message: bug fix
Parts:
- C1: footprint Jumper:SolderJumper-3_P1.3mm_Open_RoundedPad1.0x1.5mm -> Capacitor_SMD:C_0603_1608Metric_Pad1.08x0.95mm_HandSolder
Changed lines of the file:
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@@
       (effects (font (size 1.27 1.27)) (justify left))
     )
-    (property "Footprint" "Jumper:SolderJumper-3_P1.3mm_Open_RoundedPad1.0x1.5mm" (at 53.34 82.55 0)
+    (property "Footprint" "Capacitor_SMD:C_0603_1608Metric_Pad1.08x0.95mm_HandSolder" (at 53.34 82.55 0)
       (effects (font (size 1.27 1.27)) hide)
     )
