File: sync.kicad_pcb (KiCad board)
At the start: 2 copper layers, 50 x 20 mm, 5 parts, among them J1 Conn_01x04_Male, J2 Conn_01x04_Male, U1 LTC1485

Commit message: update
Parts:
- U1: footprint Package_DIP:DIP-8_W7.62mm -> Package_SO:SO-8_3.9x4.9mm_P1.27mm
- moved J1 14.4 mm to (96.8, 65.0)
- moved J2 12.3 mm to (62.6, 73.8), turned to 90 degrees
- moved U1 7.18 mm to (93.0, 73.0)
- moved C1 5.83 mm to (93.0, 69.0)
- moved R1 2.21 mm to (87.5, 73.0)
Connections:
- J1 pad 1: VCC -> unconnected-(J1-Pad1)
- J1 pad 2: GND1 -> SIGNAL
- J1 pad 3: Net-(J1-Pad3) -> VCC
- J1 pad 4: unconnected-(J1-Pad4) -> GND1
- J2 pad 1: unconnected-(J2-Pad1) -> Net-(J2-Pad1)
- J2 pad 3: Net-(J2-Pad3) -> Net-(J2-Pad1)
- J2 pad 4: unconnected-(J2-Pad4) -> Net-(J2-Pad2)
- R1 pad 1: Net-(J2-Pad3) -> Net-(J2-Pad2)
- R1 pad 2: Net-(J2-Pad2) -> Net-(J2-Pad1)
- U1 pad 4: Net-(J1-Pad3) -> SIGNAL
- U1 pad 6: Net-(J2-Pad2) -> Net-(J2-Pad1)
- U1 pad 7: Net-(J2-Pad3) -> Net-(J2-Pad2)
Routing:
- net VCC: track 35.8 -> 0.00 mm
- net Net-(J1-Pad3): track 27.0 -> 0.00 mm
- net Net-(J2-Pad2): track 17.8 -> 0.00 mm
- net GND1: track 15.9 -> 0.00 mm
- net Net-(J2-Pad3): track 15.5 -> 0.00 mm
- net (no net): vias 30 -> 0

Commit message: place route
Parts:
- moved C1 0.90 mm to (92.2, 69.5)
Connections:
- J2 pad 1: Net-(J2-Pad1) -> /D-
- J2 pad 2: Net-(J2-Pad2) -> /D+
- J2 pad 3: Net-(J2-Pad1) -> /D-
- J2 pad 4: Net-(J2-Pad2) -> /D+
- R1 pad 1: Net-(J2-Pad2) -> /D-
- R1 pad 2: Net-(J2-Pad1) -> /D+
- U1 pad 6: Net-(J2-Pad1) -> /D+
- U1 pad 7: Net-(J2-Pad2) -> /D-
Routing:
- net /D+: track 0.00 -> 37.7 mm
- net /D-: track 0.00 -> 37.4 mm
- net VCC: track 0.00 -> 17.8 mm
- net SIGNAL: track 0.00 -> 6.64 mm
- net GND1: vias 0 -> 5
- added copper zone on B.Cu, net GND1
- added copper zone on F.Cu, net GND1

Commit message: modify
Parts:
- J2: footprint Connector_JST:JST_XA_S04B-XASK-1_1x04_P2.50mm_Horizontal -> Connector_JST:JST_XA_S04B-XASK-1N-BN_1x04_P2.50mm_Horizontal
Connections:
- J2 pad 1: /D- -> /D+
- J2 pad 2: /D+ -> /D-
- J2 pad 3: /D- -> /D+
- J2 pad 4: /D+ -> /D-
Routing:
- net /D+: track 37.7 -> 37.0 mm
- net /D-: track 37.4 -> 37.5 mm, vias 0 -> 1
Changed lines of the file:
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@@
     )
   )
-  (footprint "Connector_JST:JST_XA_S04B-XASK-1_1x04_P2.50mm_Horizontal" (layer "F.Cu")
+  (footprint "Connector_JST:JST_XA_S04B-XASK-1N-BN_1x04_P2.50mm_Horizontal" (layer "F.Cu")
     (at 62.6 73.75 90)
-    (descr "JST XA series connector, S04B-XASK-1 (http://www.jst-mfg.com/product/pdf/eng/eXA1.pdf), generated with kicad-footprint-generator")
-    (tags "connector JST XA horizontal hook")
+    (descr "JST XA series connector, S04B-XASK-1N-BN (http://www.jst-mfg.com/product/pdf/eng/eXA1.pdf), generated with kicad-footprint-generator")
+    (tags "connector JST XA horizontal")
     (property "Sheetfile" "sync.kicad_sch")
     (property "Sheetname" "")
@@
     (property "ki_keywords" "connector")
     (attr through_hole)
-    (fp_text reference "J2" (at -4.5 2) (layer "F.SilkS")
-        (effects (font (size 1 1) (thickness 0.15)))
-    )
-    (fp_text value "Conn_01x04_Male" (at 3.75 10.4 90) (layer "F.Fab") hide
+    (fp_text reference "J2" (at 3.75 -4.6 90) (layer "F.SilkS")
+        (effects (font (size 1 1) (thickness 0.15)))
+    )
+    (fp_text value "Conn_01x04_Male" (at 3.75 10.4 90) (layer "F.Fab")
         (effects (font (size 1 1) (thickness 0.15)))
     )
@@
     (fp_line (start -2.61 9.31) (end 10.11 9.31)
       (stroke (width 0.12) (type solid)) (layer "F.SilkS"))
-    (fp_line (start -1.5 7.01) (end 2.15 7.01)
+    (fp_line (start -1.5 7.01) (end 9 7.01)
       (stroke (width 0.12) (type solid)) (layer "F.SilkS"))
     (fp_line (start -1.5 9.31) (end -1.5 7.01)
@@
     (fp_line (start 4.55 5.2) (end 2.95 5.2)
       (stroke (width 0.12) (type solid)) (layer "F.SilkS"))
-    (fp_line (start 5.35 7.01) (end 9 7.01)
-      (stroke (width 0.12) (type solid)) (layer "F.SilkS"))
     (fp_line (start 6.45 2) (end 6.95 2)
       (stroke (width 0.12) (type solid)) (layer "F.SilkS"))
@@
     (fp_line (start 10 9.2) (end 10 -3.4)
       (stroke (width 0.1) (type solid)) (layer "F.Fab"))
-    (pad "" np_thru_hole oval (at 3.75 6.5 90) (size 2.8 2) (drill oval 2.8 2) (layers "*.Cu" "*.Mask"))
     (pad "1" thru_hole roundrect (at 0 0 90) (size 1.7 1.95) (drill 0.95) (layers "*.Cu" "*.Mask") (roundrect_rratio 0.147059)
-      (net 6 "/D-") (pinfunction "Pin_1") (pintype "passive"))
+      (net 5 "/D+") (pinfunction "Pin_1") (pintype "passive"))
     (pad "2" thru_hole oval (at 2.5 0 90) (size 1.7 1.95) (drill 0.95) (layers "*.Cu" "*.Mask")
-      (net 5 "/D+") (pinfunction "Pin_2") (pintype "passive"))
+      (net 6 "/D-") (pinfunction "Pin_2") (pintype "passive"))
     (pad "3" thru_hole oval (at 5 0 90) (size 1.7 1.95) (drill 0.95) (layers "*.Cu" "*.Mask")
-      (net 6 "/D-") (pinfunction "Pin_3") (pintype "passive"))
+      (net 5 "/D+") (pinfunction "Pin_3") (pintype "passive"))
     (pad "4" thru_hole oval (at 7.5 0 90) (size 1.7 1.95) (drill 0.95) (layers "*.Cu" "*.Mask")
-      (net 5 "/D+") (pinfunction "Pin_4") (pintype "passive"))
-    (model "${KICAD6_3DMODEL_DIR}/Connector_JST.3dshapes/JST_XA_S04B-XASK-1_1x04_P2.50mm_Horizontal.wrl"
+      (net 6 "/D-") (pinfunction "Pin_4") (pintype "passive"))
+    (model "${KICAD6_3DMODEL_DIR}/Connector_JST.3dshapes/JST_XA_S04B-XASK-1N-BN_1x04_P2.50mm_Horizontal.wrl"
       (offset (xyz 0 0 0))
       (scale (xyz 1 1 1))
@@
   (segment (start 95.575 71.095) (end 95.575 67.825) (width 0.25) (layer "F.Cu") (net 4))
   (segment (start 94.26 66.51) (end 94.26 65) (width 0.25) (layer "F.Cu") (net 4))
-  (segment (start 66.6 72.75) (end 66.1 72.25) (width 0.25) (layer "F.Cu") (net 5))
-  (segment (start 61.25 66.25) (end 62.6 66.25) (width 0.25) (layer "F.Cu") (net 5))
-  (segment (start 64.575 72.25) (end 63.575 71.25) (width 0.25) (layer "F.Cu") (net 5))
-  (segment (start 60.5 70.5) (end 60.5 67) (width 0.25) (layer "F.Cu") (net 5))
-  (segment (start 61.25 71.25) (end 60.5 70.5) (width 0.25) (layer "F.Cu") (net 5))
+  (segment (start 63.6 72.75) (end 62.6 73.75) (width 0.25) (layer "F.Cu") (net 5))
+  (segment (start 87.5 72.175) (end 86.787499 72.175) (width 0.25) (layer "F.Cu") (net 5))
   (segment (start 90.425 72.365) (end 87.69 72.365) (width 0.25) (layer "F.Cu") (net 5))
-  (segment (start 60.5 67) (end 61.25 66.25) (width 0.25) (layer "F.Cu") (net 5))
-  (segment (start 86.212499 72.75) (end 66.6 72.75) (width 0.25) (layer "F.Cu") (net 5))
-  (segment (start 87.5 72.175) (end 86.787499 72.175) (width 0.25) (layer "F.Cu") (net 5))
-  (segment (start 63.575 71.25) (end 62.6 71.25) (width 0.25) (layer "F.Cu") (net 5))
+  (segment (start 87.69 72.365) (end 87.5 72.175) (width 0.25) (layer "F.Cu") (net 5))
   (segment (start 86.787499 72.175) (end 86.212499 72.75) (width 0.25) (layer "F.Cu") (net 5))
-  (segment (start 66.1 72.25) (end 64.575 72.25) (width 0.25) (layer "F.Cu") (net 5))
-  (segment (start 62.6 71.25) (end 61.25 71.25) (width 0.25) (layer "F.Cu") (net 5))
-  (segment (start 87.69 72.365) (end 87.5 72.175) (width 0.25) (layer "F.Cu") (net 5))
-  (segment (start 62.6 71.25) (end 63.25 71.25) (width 0.25) (layer "B.Cu") (net 5))
-  (segment (start 64.575 72.75) (end 63.575 73.75) (width 0.25) (layer "F.Cu") (net 6))
-  (segment (start 87.5 73.825) (end 86.787499 73.825) (width 0.25) (layer "F.Cu") (net 6))
-  (segment (start 86.212499 73.25) (end 66.392893 73.25) (width 0.25) (layer "F.Cu") (net 6))
-  (segment (start 66.392893 73.25) (end 65.892893 72.75) (width 0.25) (layer "F.Cu") (net 6))
-  (segment (start 63.575 73.75) (end 62.6 73.75) (width 0.25) (layer "F.Cu") (net 6))
+  (segment (start 86.212499 72.75) (end 63.6 72.75) (width 0.25) (layer "F.Cu") (net 5))
+  (segment (start 60.5 69.25) (end 61 68.75) (width 0.25) (layer "B.Cu") (net 5))
+  (segment (start 60.5 73) (end 60.5 69.25) (width 0.25) (layer "B.Cu") (net 5))
+  (segment (start 61 68.75) (end 62.6 68.75) (width 0.25) (layer "B.Cu") (net 5))
+  (segment (start 61.25 73.75) (end 60.5 73) (width 0.25) (layer "B.Cu") (net 5))
+  (segment (start 62.6 73.75) (end 61.25 73.75) (width 0.25) (layer "B.Cu") (net 5))
+  (segment (start 67.5 73.25) (end 86.212499 73.25) (width 0.25) (layer "F.Cu") (net 6))
+  (segment (start 61.25 66.25) (end 62.6 66.25) (width 0.25) (layer "F.Cu") (net 6))
+  (segment (start 86.212499 73.25) (end 86.787499 73.825) (width 0.25) (layer "F.Cu") (net 6))
+  (segment (start 60.5 70.5) (end 60.5 67) (width 0.25) (layer "F.Cu") (net 6))
+  (segment (start 61.25 71.25) (end 60.5 70.5) (width 0.25) (layer "F.Cu") (net 6))
+  (segment (start 60.5 67) (end 61.25 66.25) (width 0.25) (layer "F.Cu") (net 6))
   (segment (start 87.69 73.635) (end 87.5 73.825) (width 0.25) (layer "F.Cu") (net 6))
-  (segment (start 65.892893 72.75) (end 64.575 72.75) (width 0.25) (layer "F.Cu") (net 6))
-  (segment (start 86.787499 73.825) (end 86.212499 73.25) (width 0.25) (layer "F.Cu") (net 6))
+  (segment (start 62.6 71.25) (end 61.25 71.25) (width 0.25) (layer "F.Cu") (net 6))
+  (segment (start 67.25 73.5) (end 67.5 73.25) (width 0.25) (layer "F.Cu") (net 6))
   (segment (start 90.425 73.635) (end 87.69 73.635) (width 0.25) (layer "F.Cu") (net 6))
-  (segment (start 60.25 72.75) (end 60.25 69.5) (width 0.25) (layer "B.Cu") (net 6))
-  (segment (start 60.25 69.5) (end 61 68.75) (width 0.25) (layer "B.Cu") (net 6))
-  (segment (start 61 68.75) (end 62.6 68.75) (width 0.25) (layer "B.Cu") (net 6))
-  (segment (start 62.6 73.75) (end 61.25 73.75) (width 0.25) (layer "B.Cu") (net 6))
-  (segment (start 61.25 73.75) (end 60.25 72.75) (width 0.25) (layer "B.Cu") (net 6))
+  (segment (start 86.787499 73.825) (end 87.5 73.825) (width 0.25) (layer "F.Cu") (net 6))
+  (via (at 67.25 73.5) (size 0.8) (drill 0.4) (layers "F.Cu" "B.Cu") (net 6))
+  (segment (start 67.25 73.5) (end 66.5 73.5) (width 0.25) (layer "B.Cu") (net 6))
+  (segment (start 64.25 71.25) (end 62.6 71.25) (width 0.25) (layer "B.Cu") (net 6))
+  (segment (start 66.5 73.5) (end 64.25 71.25) (width 0.25) (layer "B.Cu") (net 6))
   (zone (net 2) (net_name "GND1") (layers "F&B.Cu") (hatch edge 0.5)
     (connect_pads (clearance 0.508))

Commit message: backup
Parts:
- added D1: ~, sync:SMA (DO-214AC), F.Cu at (83.0, 76.5)
- added D2: ~, sync:SMA (DO-214AC), F.Cu at (83.5, 66.5)
- added JP1: SolderJumper_3_Open, Jumper:SolderJumper-3_P1.3mm_Open_Pad1.0x1.5mm, F.Cu at (83.8, 70.2)
- added R2: 1K, Resistor_SMD:R_0603_1608Metric, F.Cu at (82.0, 73.2)
- C1: footprint Capacitor_SMD:C_0603_1608Metric -> Jumper:SolderJumper-3_P1.3mm_Open_RoundedPad1.0x1.5mm
- moved R1 2.02 mm to (85.5, 73.2)
Connections:
- R1 pad 2: /D+ -> Net-(JP1-B)
Routing:
- net GND1: track 0.00 -> 9.53 mm
- net /D+: track 37.0 -> 43.2 mm
- net /D-: track 37.5 -> 40.6 mm, vias 1 -> 0
- net Net-(JP1-A): track 0.00 -> 2.36 mm
- net Net-(JP1-B): track 0.00 -> 2.11 mm

Commit message: bug fix
Parts:
- C1: footprint Jumper:SolderJumper-3_P1.3mm_Open_RoundedPad1.0x1.5mm -> Capacitor_SMD:C_0603_1608Metric_Pad1.08x0.95mm_HandSolder
- D1, D2: value ~ -> 12V
- moved C1 0.75 mm to (92.2, 68.8)
Routing:
- net GND1: track 9.53 -> 8.17 mm, vias 5 -> 7
Other:
- rule pad_to_mask_clearance: 0 -> 0.1

Commit message: gerber
Parts:
- moved D1 0.90 mm to (83.8, 76.0)
- moved R1 0.71 mm to (85.0, 72.8)
- moved JP1 0.50 mm to (83.8, 69.8)
- moved R2 0.50 mm to (82.0, 72.8)
- moved D2 0.25 mm to (83.5, 66.2)
Routing:
- net GND1: track 8.17 -> 0.00 mm
- net Net-(JP1-A): track 2.36 -> 1.86 mm
